Commit message: 已实现基本轮式移动

File: source/robot_lab/data/Robots/unitree/Go2wArm_description/urdf/go2w_piper_description_NoGrip.urdf (robot description, URDF)
Before this commit: robot go2w_piper_description, 41 links, 40 joints
Links:
- link FL_foot: geometry collision cylinder length=0.045 radius=0.086; visual mesh filename=../meshes_mjc/left_wheel.stl
- link FR_foot: geometry collision cylinder length=0.045 radius=0.086; visual mesh filename=../meshes_mjc/right_wheel.stl
- link RL_foot: geometry collision cylinder length=0.045 radius=0.086; visual mesh filename=../meshes_mjc/left_wheel.stl
- link RR_foot: geometry collision cylinder length=0.045 radius=0.086; visual mesh filename=../meshes_mjc/right_wheel.stl
